File: schematics/mainboard.sch (EAGLE design)
At the start: 11 parts, among them IC2 L293D

Commit message: Switched to proper servo. Updated PCB. Did not update for new IMU
Parts:
- removed IC2: L293D, st-microelectronics:L293D
- removed STEERING: (no value), con-lstb:MA05-1
- added STEER_SERVO: (no value), con-lstb:MA03-1
Connections:
- removed net N$3: IC2.1Y, STEERING.4
- removed net N$4: IC2.2Y, STEERING.5
- removed net STEER_1: IC2.1A, U$1.A1
- removed net STEER_2: IC2.2A, U$1.A0
- removed net STEER_POS: STEERING.2, U$1.A2
- new net STEER_SIGNAL: STEER_SERVO.1, U$1.D4
- net +5V: now also STEER_SERVO.2; no longer IC2.1-2EN, IC2.VCC1, IC2.VCC2, STEERING.1
- net GND: now also STEER_SERVO.3; no longer IC2.3-4EN, IC2.3A, IC2.4A, IC2.GND1, IC2.GND2, IC2.GND3, IC2.GND4, STEERING.3
